Commit message: cool com experiment in deformable sim

File: deform/src/geo/block.urdf (robot description, URDF)
Before this commit: robot block, 1 links, 0 joints
Links:
- link blocka: geometry collision box size=0.8 0.8 0.8; visual box size=0.8 0.8 0.8

Commit message: documentation update and some cleaning

File: deform/src/geo/block.urdf (robot description, URDF)
Before this commit: robot block, 1 links, 0 joints
Links:
- link blocka: geometry collision box size=0.6 0.6 0.6; visual box size=0.6 0.6 0.6

File: deform/src/geo/block2.urdf (robot description, URDF)
Before this commit: robot block, 1 links, 0 joints
Links:
- link blocka: geometry collision box size=0.6 0.6 0.6; visual box size=0.6 0.6 0.6

Commit message: added prelim grid search

File: deform/src/geo/block.urdf (robot description, URDF)
Before this commit: robot block, 1 links, 0 joints
Links:
- link blocka: mass 1.0 -> 1.6

File: deform/src/geo/block2.urdf (robot description, URDF)
Before this commit: robot block, 1 links, 0 joints
Links:
- link blocka: mass 1.0 -> 1

Commit message: small mesh

File: deform/src/geo/block.urdf (robot description, URDF)
Before this commit: robot block, 1 links, 0 joints
Links:
- link blocka: mass 1.6 -> .08; geometry collision box size=0.06 0.06 0.06; visual box size=0.06 0.06 0.06
