Commit message: Add URDF for the frame and table

File: tamp/models/panda_table.urdf (robot description, URDF)
Before this commit: robot flat_terrain, 5 links, 4 joints
Links:
- removed link vertical_support_1
- removed link vertical_support_2
- removed link vertical_support_3
- removed link vertical_support_4
Joints:
- removed joint vertical_1_base_fixed
- removed joint vertical_2_base_fixed
- removed joint vertical_3_base_fixed
- removed joint vertical_4_base_fixed
