Commit message: Update initial block and regrasp locations

File: tamp/models/walls.urdf (robot description, URDF)
Before this commit: robot walls, 4 links, 3 joints
Joints:
- joint left_front: origin xyz=-0.767 0.6146 0.0 rpy=0 0 0 -> xyz=-0.767 0.8146 0.0 rpy=0 0 0
- joint right_front: origin xyz=-0.767 -0.6146 0.0 rpy=0 0 0 -> xyz=-0.767 -0.8146 0.0 rpy=0 0 0
